File: electronics/drive/drive.sch (EAGLE design)
At the start: 11 parts, among them IC1 MEGA8-AI, IC2 MAX1483ESA, J1 AVR_SPI_PRG_6NS

Commit message: Updating the board - More space for the programming connector - VCC connected to the programming connector - Removed the jumper wire
Connections:
- net +5V: now also J1.2
Changed lines of the file:
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@@
 <?xml version="1.0" encoding="utf-8"?>
 <!DOCTYPE eagle SYSTEM "eagle.dtd">
-<eagle version="6.2">
+<eagle version="6.5.0">
 <drawing>
 <settings>
@@
 <part name="R3" library="rcl" deviceset="R-EU_" device="R0805" value="1k"/>
 <part name="P+9" library="supply1" deviceset="+5V" device=""/>
+<part name="P+10" library="supply1" deviceset="+5V" device=""/>
 </parts>
 <sheets>
@@
 <instance part="R3" gate="G$1" x="-12.7" y="7.62" rot="R180"/>
 <instance part="P+9" gate="1" x="5.08" y="96.52"/>
+<instance part="P+10" gate="1" x="15.24" y="-30.48" rot="R270"/>
 </instances>
 <busses>
@@
 <pinref part="P+9" gate="1" pin="+5V"/>
 </segment>
+<segment>
+<pinref part="J1" gate="G$1" pin="2"/>
+<pinref part="P+10" gate="1" pin="+5V"/>
+<wire x1="12.7" y1="-30.48" x2="7.62" y2="-30.48" width="0.1524" layer="91"/>
+</segment>
 </net>
