File: electronics/drive/drive.brd (EAGLE design)
At the start: 35 x 25 mm, 11 parts, among them IC1 MEGA8-AI, IC2 MAX1483ESA, J1 AVR_SPI_PRG_6NS

Commit message: Moved the programming connector on drive board.
Now all three connectors can be connectors can be in at the same time.
Parts:
- moved J1 1.42 mm to (27.3, 10.8)
Routing:
- net RESET: track 10.6 -> 12.9 mm
- net GND: track 164.9 -> 166.7 mm
- net SCK: track 5.60 -> 4.60 mm
- net MOSI: track 18.6 -> 17.9 mm
- net +5V: track 90.5 -> 89.8 mm
Changed lines of the file:
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@@
 <attribute name="OC_NEWARK" value="90C3817" x="17.78" y="20.0025" size="1.778" layer="27" rot="R270" display="off"/>
 </element>
-<element name="J1" library="SparkFun" package="2X3-NS" value="AVR_SPI_PRG_6NS" x="26.67" y="12.065" rot="MR90"/>
+<element name="J1" library="SparkFun" package="2X3-NS" value="AVR_SPI_PRG_6NS" x="27.305" y="10.795" rot="MR90"/>
 <element name="R2" library="rcl" package="R0805" value="33k" x="10.795" y="15.875" rot="R90"/>
 <element name="R3" library="rcl" package="R0805" value="1k" x="24.13" y="3.175"/>
@@
 <vertex x="35.2425" y="25.4"/>
 </polygon>
-<wire x1="33.02" y1="3.175" x2="33.655" y2="3.81" width="0.3048" layer="1"/>
-<wire x1="33.655" y1="3.81" x2="33.655" y2="20.32" width="0.3048" layer="1"/>
-<wire x1="33.655" y1="20.32" x2="33.02" y2="20.955" width="0.3048" layer="1"/>
+<wire x1="33.02" y1="3.175" x2="33.02" y2="20.955" width="0.3048" layer="1"/>
 <wire x1="13.4874" y1="11.665" x2="12.465" y2="11.665" width="0.3048" layer="1"/>
 <wire x1="12.465" y1="11.665" x2="12.065" y2="12.065" width="0.3048" layer="1"/>
@@
 <wire x1="10.795" y1="13.335" x2="10.795" y2="13.015" width="0.4064" layer="1"/>
 <wire x1="22.0726" y1="12.465" x2="18.015" y2="12.465" width="0.3048" layer="1"/>
-<wire x1="20.8534" y1="18.0975" x2="26.3525" y2="18.0975" width="0.3048" layer="1"/>
-<wire x1="26.3525" y1="18.0975" x2="27.94" y2="16.51" width="0.3048" layer="1"/>
-<wire x1="27.94" y1="16.51" x2="27.94" y2="14.605" width="0.3048" layer="1"/>
+<wire x1="20.8534" y1="18.0975" x2="26.9875" y2="18.0975" width="0.3048" layer="1"/>
+<wire x1="28.575" y1="16.51" x2="28.575" y2="13.335" width="0.3048" layer="1"/>
 <wire x1="32.0675" y1="23.8125" x2="33.02" y2="22.86" width="0.3048" layer="1"/>
 <wire x1="33.02" y1="22.86" x2="33.02" y2="20.955" width="0.3048" layer="1"/>
 <wire x1="22.0726" y1="12.465" x2="23.26" y2="12.465" width="0.3048" layer="1"/>
-<wire x1="23.26" y1="12.465" x2="24.13" y2="13.335" width="0.3048" layer="1"/>
-<wire x1="24.13" y1="13.335" x2="26.67" y2="13.335" width="0.3048" layer="1"/>
-<wire x1="26.67" y1="13.335" x2="27.94" y2="14.605" width="0.3048" layer="1"/>
+<wire x1="27.305" y1="12.065" x2="28.575" y2="13.335" width="0.3048" layer="1"/>
+<wire x1="26.9875" y1="18.0975" x2="28.575" y2="16.51" width="0.3048" layer="1"/>
+<wire x1="27.305" y1="12.065" x2="23.66" y2="12.065" width="0.3048" layer="1"/>
+<wire x1="23.66" y1="12.065" x2="23.26" y2="12.465" width="0.3048" layer="1"/>
 </signal>
 <signal name="SENSOR">
@@
 <wire x1="30.48" y1="20.955" x2="30.48" y2="20.32" width="0.4064" layer="1"/>
 <wire x1="18.98" y1="7.7724" x2="18.98" y2="6.7375" width="0.3048" layer="1"/>
-<wire x1="31.75" y1="15.24" x2="31.75" y2="13.335" width="1.016" layer="1"/>
-<wire x1="31.75" y1="13.335" x2="31.75" y2="6.35" width="1.016" layer="1"/>
+<wire x1="31.75" y1="15.24" x2="31.75" y2="12.065" width="1.016" layer="1"/>
+<wire x1="31.75" y1="12.065" x2="31.75" y2="6.35" width="1.016" layer="1"/>
 <wire x1="18.98" y1="6.7375" x2="20.6375" y2="5.08" width="0.3048" layer="1"/>
 <wire x1="30.48" y1="5.08" x2="30.48" y2="3.175" width="1.016" layer="1"/>
@@
 <wire x1="30.48" y1="22.225" x2="30.48" y2="20.955" width="0.3048" layer="1"/>
 <contactref element="J1" pad="2"/>
-<wire x1="27.94" y1="9.525" x2="26.67" y2="10.795" width="0.3048" layer="1"/>
-<wire x1="26.67" y1="10.795" x2="26.67" y2="12.7" width="0.3048" layer="1"/>
-<wire x1="26.67" y1="12.7" x2="27.305" y2="13.335" width="0.3048" layer="1"/>
-<wire x1="27.305" y1="13.335" x2="31.75" y2="13.335" width="0.3048" layer="1"/>
+<wire x1="28.575" y1="8.255" x2="27.305" y2="9.525" width="0.3048" layer="1"/>
+<wire x1="27.305" y1="9.525" x2="27.305" y2="11.43" width="0.3048" layer="1"/>
+<wire x1="27.305" y1="11.43" x2="27.94" y2="12.065" width="0.3048" layer="1"/>
+<wire x1="27.94" y1="12.065" x2="31.75" y2="12.065" width="0.3048" layer="1"/>
 <wire x1="20.955" y1="23.1775" x2="20.955" y2="22.0091" width="0.3048" layer="1"/>
 <wire x1="20.955" y1="22.0091" x2="20.8534" y2="21.9075" width="0.3048" layer="1"/>
@@
 <contactref element="IC1" pad="17"/>
 <contactref element="J1" pad="3"/>
+<wire x1="24.765" y1="10.795" x2="26.035" y2="10.795" width="0.3048" layer="1"/>
 <wire x1="22.0726" y1="9.265" x2="23.235" y2="9.265" width="0.3048" layer="1"/>
-<wire x1="23.235" y1="9.265" x2="23.495" y2="9.525" width="0.3048" layer="1"/>
-<wire x1="23.495" y1="9.525" x2="23.495" y2="11.43" width="0.3048" layer="1"/>
-<wire x1="23.495" y1="11.43" x2="24.13" y2="12.065" width="0.3048" layer="1"/>
-<wire x1="24.13" y1="12.065" x2="25.4" y2="12.065" width="0.3048" layer="1"/>
+<wire x1="23.235" y1="9.265" x2="24.765" y2="10.795" width="0.3048" layer="1"/>
 </signal>
 <signal name="MISO">
 <contactref element="IC1" pad="16"/>
 <contactref element="J1" pad="1"/>
-<wire x1="20.58" y1="7.7724" x2="23.6474" y2="7.7724" width="0.3048" layer="1"/>
-<wire x1="23.6474" y1="7.7724" x2="25.4" y2="9.525" width="0.3048" layer="1"/>
+<wire x1="20.58" y1="7.7724" x2="25.5524" y2="7.7724" width="0.3048" layer="1"/>
+<wire x1="25.5524" y1="7.7724" x2="26.035" y2="8.255" width="0.3048" layer="1"/>
 </signal>
 <signal name="MOSI">
@@
 <contactref element="J1" pad="4"/>
 <wire x1="19.78" y1="6.89" x2="19.78" y2="7.7724" width="0.3048" layer="1"/>
-<wire x1="19.78" y1="6.89" x2="20.32" y2="6.35" width="0.3048" layer="1"/>
-<wire x1="20.32" y1="6.35" x2="28.575" y2="6.35" width="0.3048" layer="1"/>
-<wire x1="28.575" y1="6.35" x2="30.48" y2="8.255" width="0.3048" layer="1"/>
-<wire x1="30.48" y1="8.255" x2="30.48" y2="11.43" width="0.3048" layer="1"/>
-<wire x1="30.48" y1="11.43" x2="29.845" y2="12.065" width="0.3048" layer="1"/>
-<wire x1="29.845" y1="12.065" x2="27.94" y2="12.065" width="0.3048" layer="1"/>
+<wire x1="19.78" y1="6.89" x2="20.955" y2="5.715" width="0.3048" layer="1"/>
+<wire x1="20.955" y1="5.715" x2="29.21" y2="5.715" width="0.3048" layer="1"/>
+<wire x1="29.21" y1="5.715" x2="30.48" y2="6.985" width="0.3048" layer="1"/>
+<wire x1="30.48" y1="6.985" x2="30.48" y2="10.16" width="0.3048" layer="1"/>
+<wire x1="30.48" y1="10.16" x2="29.845" y2="10.795" width="0.3048" layer="1"/>
+<wire x1="29.845" y1="10.795" x2="28.575" y2="10.795" width="0.3048" layer="1"/>
 </signal>
 <signal name="RESET">
@@
 <wire x1="17.78" y1="14.605" x2="20.32" y2="14.605" width="0.3048" layer="1"/>
 <wire x1="20.32" y1="14.605" x2="21.59" y2="15.875" width="0.3048" layer="1"/>
-<wire x1="21.59" y1="15.875" x2="24.13" y2="15.875" width="0.3048" layer="1"/>
-<wire x1="24.13" y1="15.875" x2="25.4" y2="14.605" width="0.3048" layer="1"/>
+<wire x1="21.59" y1="15.875" x2="25.4" y2="15.875" width="0.3048" layer="1"/>
+<wire x1="26.035" y1="15.24" x2="26.035" y2="13.335" width="0.3048" layer="1"/>
+<wire x1="26.035" y1="15.24" x2="25.4" y2="15.875" width="0.3048" layer="1"/>
 </signal>
 <signal name="D+">
